File: KiCAD/vreg-dac-lt3014/vreg-dac-lt3014.kicad_pcb (KiCad board)
At the start: 2 copper layers, 28 parts, among them J1 Conn_01x02, J2 Conn_01x02, J3 Conn_01x02, J4 Conn_01x05, Q1 NMOS, Q2 NMOS, U1 LT3014xS5, U3 INA200D, U4 AD5270

Commit message: working on layout
Parts:
- removed Q1, Q2: NMOS, Package_TO_SOT_SMD:SOT-23
- added C10: ~, Capacitor_SMD:C_0603_1608Metric_Pad1.08x0.95mm_HandSolder, F.Cu at (100.3, 54.6)
- added D2: LED, LED_SMD:LED_0603_1608Metric_Pad1.05x0.95mm_HandSolder, F.Cu at (100.1, 47.0)
- added D3: LED, LED_SMD:LED_0603_1608Metric_Pad1.05x0.95mm_HandSolder, F.Cu at (95.9, 105.4)
- added D4: LED, LED_SMD:LED_0603_1608Metric_Pad1.05x0.95mm_HandSolder, F.Cu at (103.5, 105.4)
- added H1: MountingHole, MountingHole:MountingHole_4.3mm_M4, F.Cu at (87.6, 48.3)
- added H2: MountingHole, MountingHole:MountingHole_4.3mm_M4, F.Cu at (142.2, 48.3)
- added H3: MountingHole, MountingHole:MountingHole_4.3mm_M4, F.Cu at (87.6, 108.0)
- added H4: MountingHole, MountingHole:MountingHole_4.3mm_M4, F.Cu at (142.2, 108.0)
- added J5: Conn_01x04, Connector_PinHeader_2.54mm:PinHeader_1x04_P2.54mm_Vertical, F.Cu at (98.6, 110.7)
- added Q3: BSS138, Package_TO_SOT_SMD:SOT-23, F.Cu at (118.9, 51.4)
- added Q4: BSS138, Package_TO_SOT_SMD:SOT-23, F.Cu at (126.4, 66.0)
- added Q5: BSS138, Package_TO_SOT_SMD:SOT-23, F.Cu at (119.4, 61.6)
- added R10: 10.0k 1%, Resistor_SMD:R_0603_1608Metric_Pad0.98x0.95mm_HandSolder, F.Cu at (129.5, 62.2)
- added R11: 210k, Resistor_SMD:R_0603_1608Metric_Pad0.98x0.95mm_HandSolder, F.Cu at (104.8, 57.5)
- added R12: 140k, Resistor_SMD:R_0603_1608Metric_Pad0.98x0.95mm_HandSolder, F.Cu at (104.8, 60.6)
- added R13: 0R, Resistor_SMD:R_0603_1608Metric_Pad0.98x0.95mm_HandSolder, F.Cu at (95.9, 58.4)
- added R14: 0R, Resistor_SMD:R_0603_1608Metric_Pad0.98x0.95mm_HandSolder, F.Cu at (100.3, 58.4)
- added R15: 10k, Resistor_SMD:R_0603_1608Metric_Pad0.98x0.95mm_HandSolder, F.Cu at (124.0, 61.6)
- added R16: 100k, Resistor_SMD:R_0603_1608Metric_Pad0.98x0.95mm_HandSolder, F.Cu at (125.7, 71.1)
- added R17: 1.5k, Resistor_SMD:R_0603_1608Metric_Pad0.98x0.95mm_HandSolder, F.Cu at (99.7, 105.4)
- added R18: 1.5k, Resistor_SMD:R_0603_1608Metric_Pad0.98x0.95mm_HandSolder, F.Cu at (107.3, 105.4)
- added R8: 1.5k, Resistor_SMD:R_0603_1608Metric_Pad0.98x0.95mm_HandSolder, F.Cu at (100.1, 50.2)
- added R9: 200k 1%, Resistor_SMD:R_0603_1608Metric_Pad0.98x0.95mm_HandSolder, F.Cu at (129.5, 59.7)
- added TP10: GND, my_tp:tp_SMT_label2, F.Cu at (139.7, 73.7)
- added TP5: VIN60, my_tp:tp_SMT_label2, F.Cu at (90.8, 57.1)
- added TP6: VSENSE, my_tp:tp_SMT_label2, F.Cu at (135.8, 57.7)
- added TP7: IMON, my_tp:tp_SMT_label2, F.Cu at (107.3, 47.6)
- added TP8: CMP, my_tp:tp_SMT_label2, F.Cu at (113.7, 47.6)
- added TP9: GND, my_tp:tp_SMT_label2, F.Cu at (92.1, 74.9)
- J4: value Conn_01x05 -> Conn_01x08; footprint Connector_PinHeader_2.54mm:PinHeader_1x05_P2.54mm_Vertical -> Connector_PinHeader_2.54mm:PinHeader_1x08_P2.54mm_Vertical
- R1: value 3 -> 3.00 1%
- TP1: value TestPoint -> DPOT; footprint TestPoint:TestPoint_THTPad_D2.0mm_Drill1.0mm -> my_tp:tp_SMT_label2
- TP2: value TestPoint -> VR_ADJ; footprint TestPoint:TestPoint_THTPad_D2.0mm_Drill1.0mm -> my_tp:tp_SMT_label2
- TP3: value TestPoint -> VR_IN; footprint TestPoint:TestPoint_THTPad_D2.0mm_Drill1.0mm -> my_tp:tp_SMT_label2
- TP4: value TestPoint -> OUTPUT; footprint TestPoint:TestPoint_THTPad_D2.0mm_Drill1.0mm -> my_tp:tp_SMT_label2
- U3: value INA200D -> INA201
- moved D1 81.0 mm to (124.5, 47.0), turned to 180 degrees
- moved TP4 73.7 mm to (139.1, 64.1)
- moved R7 60.4 mm to (132.1, 66.7)
- moved R6 59.6 mm to (124.5, 49.5), turned to 180 degrees
- moved C8 58.9 mm to (121.5, 66.0), turned to 180 degrees
- moved R5 57.1 mm to (124.5, 52.1), turned to 180 degrees
- moved TP2 55.5 mm to (119.1, 71.9)
- moved C7 48.6 mm to (110.8, 64.0), turned to 180 degrees
- moved C6 47.9 mm to (112.7, 70.6), turned to 180 degrees
- moved R4 46.5 mm to (113.7, 52.1)
- moved TP1 44.4 mm to (105.3, 73.5)
- moved TP3 35.9 mm to (101.0, 66.7)
- moved R1 24.2 mm to (95.9, 62.2), turned to 0 degrees
- moved C9 20.3 mm to (104.8, 54.6), turned to 180 degrees
- moved J1 19.1 mm to (144.8, 59.7)
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Connections:
- A1 pad 1: unconnected-(A1-GPIO0-Pad1) -> /LED1
- A1 pad 13: Net-(A1-GND-Pad13) -> GND
- A1 pad 18: Net-(A1-GND-Pad13) -> GND
- A1 pad 2: unconnected-(A1-GPIO1-Pad2) -> /LED2
- A1 pad 22: unconnected-(A1-GPIO17-Pad22) -> /~{SYNC}
- A1 pad 23: Net-(A1-GND-Pad13) -> GND
- A1 pad 24: unconnected-(A1-GPIO18-Pad24) -> /SCLK
- A1 pad 25: unconnected-(A1-GPIO19-Pad25) -> /SDA
- A1 pad 26: unconnected-(A1-GPIO20-Pad26) -> /RESET
- A1 pad 27: unconnected-(A1-GPIO21-Pad27) -> /SHDN
- A1 pad 28: Net-(A1-GND-Pad13) -> GND
- A1 pad 29: unconnected-(A1-GPIO22-Pad29) -> /SHUTDOWN
- A1 pad 3: Net-(A1-GND-Pad13) -> GND
- A1 pad 31: unconnected-(A1-GPIO26_ADC0-Pad31) -> /IMON
- A1 pad 32: unconnected-(A1-GPIO27_ADC1-Pad32) -> /VSENSE
- A1 pad 33: unconnected-(A1-AGND-Pad33) -> GND
- A1 pad 36: unconnected-(A1-3V3-Pad36) -> +3.3V
- A1 pad 38: Net-(A1-GND-Pad13) -> GND
- A1 pad 6: unconnected-(A1-GPIO4-Pad6) -> /GP0/TX
- A1 pad 7: unconnected-(A1-GPIO5-Pad7) -> /GP1/RX
- A1 pad 8: Net-(A1-GND-Pad13) -> GND
- A1 pad 9: unconnected-(A1-GPIO6-Pad9) -> /GP2
- C4 pad 1: Net-(J2-Pin_1) -> Net-(U1-VIN)
- C5 pad 1: Net-(U1-VOUT) -> Net-(J1-Pin_1)
- D1 pad 1: Net-(D1-K) -> /SHDN
- J4 pad 2: /DIN -> /SDA
- J4 pad 5: GND -> /RESET
- R1 pad 1: Net-(U1-VOUT) -> Net-(J2-Pin_1)
- R1 pad 2: Net-(J1-Pin_1) -> Net-(U1-VIN)
- R2 pad 1: Net-(U1-VOUT) -> Net-(J1-Pin_1)
- R5 pad 2: Net-(D1-K) -> /SHDN
- TP3 pad 1: Net-(U1-VOUT) -> Net-(U1-VIN)
- U1 pad 1: Net-(J2-Pin_1) -> Net-(U1-VIN)
- U1 pad 3: Net-(D1-K) -> /SHDN
- U1 pad 5: Net-(U1-VOUT) -> Net-(J1-Pin_1)
- U3 pad 2: Net-(U3-CMP_{IN}) -> /IMON
- U3 pad 5: unconnected-(U3-~{RESET}-Pad5) -> Net-(Q5-D)
- U3 pad 7: Net-(J1-Pin_1) -> Net-(U3-V_{IN-})
- U3 pad 8: Net-(U1-VOUT) -> Net-(U3-V_{IN+})
- U4 pad 8: /DIN -> /SDA
Routing:
- net /VSENSE: track 0.00 -> 51.9 mm, vias 0 -> 2
- net /IMON: track 0.00 -> 42.6 mm, vias 0 -> 1
- net /RESET: track 0.00 -> 38.1 mm, vias 0 -> 1
- net Net-(U1-VIN): track 0.00 -> 38.0 mm
- net /~{SYNC}: track 0.00 -> 35.2 mm
- net /SCLK: track 0.00 -> 33.1 mm, vias 0 -> 1
- net Net-(J1-Pin_1): track 0.00 -> 32.1 mm
- net /SDA: track 0.00 -> 30.0 mm, vias 0 -> 1
- net Net-(U3-V_{IN+}): track 0.00 -> 21.5 mm
- net Net-(U1-ADJ): track 0.00 -> 19.6 mm
- net GND: track 0.00 -> 18.9 mm, vias 0 -> 13
- net Net-(U3-V_{IN-}): track 0.00 -> 18.6 mm
- net Net-(J2-Pin_1): track 0.00 -> 16.8 mm
- net Net-(Q3-G): track 0.00 -> 16.0 mm
- net Net-(Q5-D): track 0.00 -> 13.5 mm, vias 0 -> 2
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- added copper zone on In2.Cu, net +3.3V
- added copper zone on In1.Cu, net GND
Other:
- board outline added: 64.8 x 69.8 mm
- copper layers 2 -> 4
- board text added: "3.3V"
- board text added: "60V"
- board text added: "GPIO/UART"
- board text added: "NN SiPM HV trim Test Board - ESH V1.0 2025-05"
- board text added: "SHUTDOWN"
- board text added: "VOUT"

Commit message: new placement
Parts:
- added JP1: Jumper_2_Open, Connector_PinHeader_2.54mm:PinHeader_1x02_P2.54mm_Vertical, F.Cu at (107.1, 75.9)
- D1, D2, D3, D4: footprint LED_SMD:LED_0603_1608Metric_Pad1.05x0.95mm_HandSolder -> my_smt_led:my_SMT_0603
- moved TP1 32.3 mm to (135.3, 61.5)
- moved TP7 28.2 mm to (101.1, 75.1)
- moved TP8 24.8 mm to (101.1, 69.0)
- moved D2 24.1 mm to (86.3, 66.8), turned to 0 degrees
- moved R7 22.8 mm to (109.7, 62.2)
- moved TP3 19.8 mm to (104.9, 47.2)
- moved TP4 17.9 mm to (133.5, 47.1)
- moved R2 17.4 mm to (129.8, 55.7), turned to 180 degrees
- moved R8 17.2 mm to (95.7, 66.9), turned to 0 degrees
- moved R16 16.3 mm to (109.5, 69.5)
- moved R15 15.7 mm to (109.5, 67.5)
- moved TP2 15.6 mm to (125.0, 57.4)
- moved R3 14.9 mm to (129.8, 57.7), turned to 0 degrees
- moved C7 14.3 mm to (124.9, 61.6), turned to 0 degrees
- moved C6 12.4 mm to (124.8, 68.2)
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Connections:
- A1 pad 36: +3.3V -> Net-(A1-3V3)
Routing:
- net /VSENSE: track 51.9 -> 0.00 mm, vias 2 -> 0
- net /IMON: track 42.6 -> 0.00 mm, vias 1 -> 0
- net /RESET: track 38.1 -> 0.00 mm, vias 1 -> 0
- net Net-(U1-VIN): track 38.0 -> 0.00 mm
- net /~{SYNC}: track 35.2 -> 0.00 mm
- net /SCLK: track 33.1 -> 0.00 mm, vias 1 -> 0
- net Net-(J1-Pin_1): track 32.1 -> 0.00 mm
- net /SDA: track 30.0 -> 0.00 mm, vias 1 -> 0
- net Net-(U3-V_{IN+}): track 21.5 -> 0.00 mm
- net Net-(U1-ADJ): track 19.6 -> 0.00 mm
- net GND: track 18.9 -> 0.00 mm, vias 13 -> 0
- net Net-(U3-V_{IN-}): track 18.6 -> 0.00 mm
- net Net-(J2-Pin_1): track 16.8 -> 0.00 mm
- net Net-(Q3-G): track 16.0 -> 0.00 mm
- net Net-(Q5-D): track 13.5 -> 0.00 mm, vias 2 -> 0
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