File: KiCAD/lt3014-test/lt3014-test.kicad_pcb (KiCad board)
At the start: 4 copper layers, 64.8 x 69.8 mm, 56 parts, among them J1 Conn_01x02, J2 Conn_01x02, J3 Conn_01x02, J4 Conn_01x08, J5 Conn_01x04, Q3 BSS138, Q4 BSS138, Q5 BSS138, U1 LT3014xS5, U3 INA201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

Commit message: candidate V1.0 LT3014 board
Parts:
- moved R5 1.55 mm to (114.3, 54.5), turned to 0 degrees
- moved R6 1.24 mm to (114.3, 49.1), turned to 0 degrees
- turned R7 to 180 degrees
Routing:
- net /VSENSE: track 0.00 -> 57.5 mm, vias 0 -> 1
- net /SHDN: track 0.00 -> 54.9 mm, vias 0 -> 2
- net /SCLK: track 0.00 -> 50.5 mm
- net /RESET: track 0.00 -> 42.9 mm
- net /SHUTDOWN: track 0.00 -> 41.8 mm
- net /~{SYNC}: track 0.00 -> 37.6 mm
- net Net-(J1-Pin_1): track 0.00 -> 37.4 mm
- net /IMON: track 0.00 -> 36.7 mm
- net /SDA: track 0.00 -> 36.1 mm, vias 0 -> 2
- net Net-(U1-VIN): track 0.00 -> 31.3 mm
- net GND: track 0.00 -> 26.5 mm, vias 0 -> 18
- net Net-(J2-Pin_1): track 0.00 -> 23.2 mm
- net Net-(Q3-G): track 0.00 -> 21.2 mm
- net /LED2: track 0.00 -> 18.2 mm, vias 0 -> 1
- net Net-(U4-A): track 0.00 -> 17.8 mm
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Other:
- board text added: "SiPM HV Control Test Board - ESH V1.0 2025-05"
- board text removed: "NN SiPM HV trim Test Board - ESH V1.0 2025-05"

Commit message: small tweaks before V1.0 fab
Parts:
- C4, C7: value 1uF -> 1.0uF
- R15, R5: value 10k -> 10.0k 1%
Connections:
- A1 pad 21: unconnected-(A1-GPIO16-Pad21) -> /SDO
- J4 pad 7: unconnected-(J4-Pin_7-Pad7) -> /SDO
- R7 pad 2: GND -> +3.3V
- U4 pad 7: unconnected-(U4-SDO-Pad7) -> /SDO
Routing:
- net /SDO: track 0.00 -> 36.3 mm, vias 0 -> 3
- net GND: track 26.5 -> 25.4 mm, vias 18 -> 17
- net +3.3V: track 9.65 -> 10.7 mm, vias 9 -> 10
Other:
- board text added: "SiPM HV Control Test Board - ESH V1.0a 2025-05"
- board text removed: "SiPM HV Control Test Board - ESH V1.0 2025-05"
