File: KiCAD/lt3014-test/lt3014-test.kicad_sch (KiCad schematic)
At the start: 56 parts, among them J1 Conn_01x02, J2 Conn_01x02, J3 Conn_01x02, J4 Conn_01x08, J5 Conn_01x04, Q3 BSS138, Q4 BSS138, Q5 BSS138, U1 LT3014xS5, U3 INA201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

Commit message: candidate V1.0 LT3014 board
Other:
- note added: "1.0"
- note added: "2025-05"
- note added: "Optional filter"
- note added: "SiPM Voltage Regulator"
Changed lines of the file:
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@@
 		(effects
 			(font
-				(size 1.27 1.27)
+				(size 1.905 1.905)
 			)
 		)
@@
 		)
 	)
-	(text "60V Input"
+	(text "2025-05"
 		(exclude_from_sim no)
-		(at 21.336 83.312 0)
+		(at 195.834 199.136 0)
 		(effects
 			(font
 				(size 1.27 1.27)
+			)
+		)
+	)
+	(text "1.0"
+		(exclude_from_sim no)
+		(at 254 199.136 0)
+		(effects
+			(font
+				(size 1.27 1.27)
+			)
+		)
+	)
+	(text "60V Input"
+		(exclude_from_sim no)
+		(at 23.876 79.502 0)
+		(effects
+			(font
+				(size 1.905 1.905)
+			)
+		)
+	)
+	(text "SiPM Voltage Regulator"
+		(exclude_from_sim no)
+		(at 184.15 176.022 0)
+		(effects
+			(font
+				(size 2.54 2.54)
 			)
 		)
@@
 		(effects
 			(font
+				(size 1.27 1.27)
+			)
+		)
+	)
+	(text "Optional filter"
+		(exclude_from_sim no)
+		(at 106.934 61.214 0)
+		(effects
+			(font

Commit message: ordering
Parts:
- A1: CatNo (none) -> 2648-SC0917-ND; MfgNo (none) -> SC0917
- C4, C7: value 1uF -> 1.0uF; CatNo (none) -> 1276-1946-1-ND; MfgNo (none) -> CL10B105KP8NNNC
- C5: CatNo (none) -> 1276-1946-1-ND; MfgNo (none) -> CL10B105KP8NNNC
- C6, C9: CatNo (none) -> 399-C0603C103M4REC7411CT-ND; MfgNo (none) -> C0603C103M4REC7411
- D1, D2, D3, D4: CatNo (none) -> 3147-B19Y1USD-20C000113U1930CT-ND; MfgNo (none) -> B19Y1USD-20C000113U1930
- H1, H2, H3, H4, JP1, TP1, TP10, TP2, TP3, TP4, TP5, TP6, TP7, TP8, TP9: now not fitted
- J1, J2, J3: CatNo (none) -> SAM10844-ND; MfgNo (none) -> TSW-102-07-F-S
- J4: CatNo (none) -> 609-3257-ND; MfgNo (none) -> 68000-208HLF
- J5: CatNo (none) -> 609-3255-ND; MfgNo (none) -> 68000-204HLF
- Q3, Q4, Q5: MfgNo (none) -> BSS138
- R1: CatNo (none) -> RMCF0603FT3R00CT-ND; MfgNo (none) -> RMCF0603FT3R00
- R10: CatNo (none) -> 311-10.0KHRCT-ND; MfgNo (none) -> RC0603FR-0710KL
- R11: CatNo (none) -> 311-210KHRCT-ND; MfgNo (none) -> RC0603FR-07210KL
- R12: CatNo (none) -> 311-140KHRCT-ND; MfgNo (none) -> RC0603FR-07140KL
- R13, R14: CatNo (none) -> 311-0.0GRCT-ND; MfgNo (none) -> RC0603JR-070RL
- R15, R5: value 10k -> 10.0k 1%; CatNo (none) -> 311-10.0KHRCT-ND; MfgNo (none) -> RC0603FR-0710KL
- R16, R7, R9: CatNo (none) -> 311-100KHRCT-ND; MfgNo (none) -> RC0603FR-07100KL
- R17, R18, R6, R8: CatNo (none) -> YAG1570CT-ND; MfgNo (none) -> RT0603BRD071K5L
- R2: CatNo (none) -> RMCF0603FT2M49CT-ND; MfgNo (none) -> RMCF0603FT2M49
- R3: CatNo (none) -> 13-RT0603BRD0750KLCT-ND; MfgNo (none) -> RT0603BRD0750KL
- R4: CatNo (none) -> YAG1676CT-ND; MfgNo (none) -> RT0603BRD074K7L
- U1: CatNo (none) -> LT3014ES5#TRPBFCT-ND; MfgNo (none) -> LT3014ES5#TRPBF
- U3: MfgNo (none) -> INA201AIDR
- U4: CatNo (none) -> 505-AD5270BRMZ-50-ND; MfgNo (none) -> AD5270BRMZ-50
Other:
- note added: "3.3V from RPI"
- note added: "50K 1024 taps"
- note added: "Misc LEDs"
- note added: "Power LED"
- note added: "Shutdown LED"
- note added: "UART / GPIO"
- moved on the sheet: D3, D4, J5, R17, R18

Commit message: small tweaks before V1.0 fab
Connections:
- net +3.3V: now also R7.2
- net GND: no longer R7.2
- net SDO: now reaches U4.7 (SDO)
- net SDO: now also A1.21 (GPIO16), J4.7 (Pin_7)
Other:
- note added: "1.0a"
- note added: "2025-05-12 Edits per BZ"
- note removed: "1.0"
Changed lines of the file:
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@@
 		)
 	)
+	(text "2025-05-12 Edits per BZ"
+		(exclude_from_sim no)
+		(at 237.998 169.926 0)
+		(effects
+			(font
+				(size 1.27 1.27)
+			)
+		)
+	)
 	(text "OUTPUT"
 		(exclude_from_sim no)
@@
 		)
 	)
-	(text "1.0"
+	(text "1.0a"
 		(exclude_from_sim no)
 		(at 254 199.136 0)
@@
 	)
 	(junction
-		(at 133.35 161.29)
-		(diameter 0)
-		(color 0 0 0 0)
-	)
-	(junction
 		(at 172.72 102.87)
 		(diameter 0)
@@
 	(wire
 		(pts
-			(xy 133.35 156.21) (xy 133.35 161.29)
-		)
-		(stroke
-			(width 0)
-			(type default)
-		)
-	)
-	(wire
-		(pts
 			(xy 133.35 41.91) (xy 133.35 88.9)
 		)
@@
 	(wire
 		(pts
-			(xy 125.73 83.82) (xy 142.24 83.82)
+			(xy 121.92 144.78) (xy 105.41 144.78)
 		)
 		(stroke
@@
 	(wire
 		(pts
-			(xy 140.97 184.15) (xy 140.97 186.69)
+			(xy 125.73 83.82) (xy 142.24 83.82)
 		)
 		(stroke
@@
 	(wire
 		(pts
-			(xy 17.78 156.21) (xy 27.94 156.21)
+			(xy 140.97 184.15) (xy 140.97 186.69)
 		)
 		(stroke
@@
 	(wire
 		(pts
-			(xy 119.38 161.29) (xy 133.35 161.29)
+			(xy 17.78 156.21) (xy 27.94 156.21)
 		)
 		(stroke
@@
 	(wire
 		(pts
+			(xy 105.41 165.1) (xy 119.38 165.1)
+		)
+		(stroke
+			(width 0)
+			(type default)
+		)
+	)
+	(wire
+		(pts
 			(xy 105.41 29.21) (xy 105.41 35.56)
 		)
@@
 	(wire
 		(pts
+			(xy 139.7 139.7) (xy 121.92 139.7)
+		)
+		(stroke
+			(width 0)
+			(type default)
+		)
+	)
+	(wire
+		(pts
 			(xy 55.88 22.86) (xy 73.66 22.86)
 		)
@@
 	(wire
 		(pts
+			(xy 121.92 139.7) (xy 121.92 144.78)
+		)
+		(stroke
+			(width 0)
+			(type default)
+		)
+	)
+	(wire
+		(pts
 			(xy 93.98 189.23) (xy 102.87 189.23)
 		)
@@
 	(wire
 		(pts
-			(xy 133.35 161.29) (xy 133.35 163.83)
+			(xy 133.35 156.21) (xy 133.35 163.83)
 		)
 		(stroke
@@
 	(wire
 		(pts
+			(xy 73.66 143.51) (xy 85.09 143.51)
+		)
+		(stroke
+			(width 0)
+			(type default)
+		)
+	)
+	(wire
+		(pts
 			(xy 78.74 80.01) (xy 78.74 83.82)
 		)
@@
 	(wire
 		(pts
+			(xy 119.38 161.29) (xy 119.38 165.1)
+		)
+		(stroke
+			(width 0)
+			(type default)
+		)
+	)
+	(wire
+		(pts
 			(xy 242.57 35.56) (xy 242.57 38.1)
 		)
@@
 		)
 	)
+	(label "SDO"
+		(at 77.47 143.51 0)
+		(effects
+			(font
+				(size 1.27 1.27)
+			)
+			(justify left bottom)
+		)
+	)
 	(label "LED1"
 		(at 128.27 173.99 90)
@@
 		)
 	)
+	(label "SDO"
+		(at 110.49 144.78 0)
+		(effects
+			(font
+				(size 1.27 1.27)
+			)
+			(justify left bottom)
+		)
+	)
 	(label "VSENSE"
 		(at 208.28 87.63 0)
@@
 					(unit 1)
 				)
+			)
+		)
+	)
+	(symbol
+		(lib_id "power:+3.3V")
+		(at 105.41 165.1 0)
+		(unit 1)
+		(exclude_from_sim no)
+		(in_bom yes)
+		(on_board yes)
+		(dnp no)
+		(fields_autoplaced yes)
+		(property "Reference" "#PWR01"
+			(at 105.41 168.91 0)
+			(effects
+				(font
+					(size 1.27 1.27)
+				)
+				(hide yes)
+			)
+		)
+		(property "Value" "+3.3V"
+			(at 105.41 160.02 0)
+			(effects
+				(font
+					(size 1.27 1.27)
+				)
+			)
+		)
+		(property "Footprint" ""
+			(at 105.41 165.1 0)
+			(effects
+				(font
+					(size 1.27 1.27)
+				)
+				(hide yes)
+			)
+		)
+		(property "Datasheet" ""
+			(at 105.41 165.1 0)
+			(effects
+				(font
+					(size 1.27 1.27)
+				)
+				(hide yes)
+			)
+		)
+		(property "Description" "Power symbol creates a global label with name \"+3.3V\""
+			(at 105.41 165.1 0)
+			(effects
+				(font
+					(size 1.27 1.27)
+				)
+				(hide yes)
+			)
+		)
+		(pin "1"
+		)
+		(instances
+			(project "lt3014-test"
+				(path "/952a2494-dc5e-4846-8ac3-c813f939709c"
+					(reference "#PWR01")
+					(unit 1)
+				)

Commit message: readme, schematic  notes
Parts:
- C4, C5, C7: value 1.0uF -> 1.0uF 100V; CatNo 1276-1946-1-ND -> 490-GRM188D72A105ME01WCT-ND; MfgNo CL10B105KP8NNNC -> GRM188D72A105ME01W
Other:
- note added: "2.0"
- note added: "2025-05-12 Edits per BZ -- As built Rev 1.0 -- 2025-06-04 Change P/N for C4, C5 for 100V"
- note removed: "1.0a"
- note removed: "2025-05-12 Edits per BZ"
Changed lines of the file:
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@@
 		)
 	)
-	(text "2025-05-12 Edits per BZ"
+	(text "2025-05-12 Edits per BZ\n  -- As built Rev 1.0 --\n\n2025-06-04 Change P/N for C4, C5 for 100V"
 		(exclude_from_sim no)
-		(at 237.998 169.926 0)
+		(at 206.502 156.21 0)
 		(effects
 			(font
 				(size 1.27 1.27)
 			)
+			(justify left)
 		)
 	)
@@
 		)
 	)
-	(text "1.0a"
+	(text "2.0"
 		(exclude_from_sim no)
 		(at 254 199.136 0)
@@
 			)
 		)
-		(property "Value" "1.0uF"
+		(property "Value" "1.0uF 100V"
 			(at 163.83 149.8599 0)
 			(effects
@@
 			)
 		)
-		(property "CatNo" "1276-1946-1-ND"
+		(property "CatNo" "490-GRM188D72A105ME01WCT-ND"
 			(at 167.64 148.59 0)
 			(effects
@@
 			)
 		)
-		(property "MfgNo" "CL10B105KP8NNNC"
+		(property "MfgNo" "GRM188D72A105ME01W"
 			(at 167.64 148.59 0)
 			(effects
@@
 			)
 		)
-		(property "Value" "1.0uF"
+		(property "Value" "1.0uF 100V"
 			(at 195.58 87.6299 0)
 			(effects
@@
 			)
 		)
-		(property "MfgNo" "CL10B105KP8NNNC"
+		(property "MfgNo" "GRM188D72A105ME01W"
 			(at 191.77 86.36 0)
 			(effects
@@
 			)
 		)
-		(property "CatNo" "1276-1946-1-ND"
+		(property "CatNo" "490-GRM188D72A105ME01WCT-ND"
 			(at 191.77 86.36 0)
 			(effects
@@
 			)
 		)
-		(property "Value" "1.0uF"
+		(property "Value" "1.0uF 100V"
 			(at 129.54 91.4399 0)
 			(effects
@@
 			)
 		)
-		(property "CatNo" "1276-1946-1-ND"
+		(property "CatNo" "490-GRM188D72A105ME01WCT-ND"
 			(at 125.73 90.17 0)
 			(effects
@@
 			)
 		)
-		(property "MfgNo" "CL10B105KP8NNNC"
+		(property "MfgNo" "GRM188D72A105ME01W"
 			(at 125.73 90.17 0)
 			(effects
