File: KiCAD/sipm-hv-splitter/sipm-hv-splitter.kicad_pcb (KiCad board)
At the start: 6 copper layers, 63.5 x 33 mm, 133 parts, among them J1 Conn_02x18_Odd_Even, J2 Conn_02x17_Odd_Even, J3 -OMIT-, Q1 BSS138, Q2 BSS138, Q3 BSS138, U1 ATmega328-M, U10 OPA810xDCK, U11 OPA810xDCK, U12 OPA810xDCK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

Commit message: routing complete
Parts:
- moved C16 0.64 mm to (98.2, 53.0)
- moved C17 0.64 mm to (98.2, 56.9)
- moved C18 0.64 mm to (98.2, 60.6)
- moved C19 0.64 mm to (98.2, 64.4)
- moved C20 0.64 mm to (98.2, 68.2)
- moved C21 0.64 mm to (98.2, 72.0)
- moved C22 0.64 mm to (98.2, 75.8)
- moved C23 0.64 mm to (98.2, 79.8)
- moved C24 0.64 mm to (98.2, 54.8)
- moved C25 0.64 mm to (98.2, 58.7)
- moved C26 0.64 mm to (98.2, 62.4)
- moved C27 0.64 mm to (98.2, 66.2)
- moved C28 0.64 mm to (98.2, 70.0)
- moved C29 0.64 mm to (98.2, 73.8)
- moved C30 0.64 mm to (98.2, 77.6)
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Connections:
- J1 pad 28: unconnected-(J1-Pin_28-Pad28) -> /TIA_6/SIPM_K
Routing:
- net /SIG_1: track 0.00 -> 44.8 mm, vias 0 -> 2
- net /SIG_7: track 0.00 -> 44.3 mm, vias 0 -> 2
- net /SIG_0: track 0.00 -> 44.1 mm, vias 0 -> 2
- net /SIG_6: track 0.00 -> 43.8 mm, vias 0 -> 2
- net /SIG_2: track 0.00 -> 43.8 mm, vias 0 -> 2
- net /SIG_5: track 0.00 -> 43.3 mm, vias 0 -> 2
- net /SIG_3: track 0.00 -> 43.3 mm, vias 0 -> 2
- net /SIG_4: track 0.00 -> 42.9 mm, vias 0 -> 2
- net GND: track 91.9 -> 117.1 mm, vias 69 -> 78
- net -24V: track 19.1 -> 34.5 mm, vias 8 -> 16
- net +12V: track 9.34 -> 23.4 mm, vias 10 -> 17
- net /TIA_6/SIPM_K: track 5.06 -> 14.8 mm
- net /DET_1: track 10.8 -> 20.4 mm
- net /TIA_5/SIPM_K: track 5.06 -> 12.8 mm
- net /DET_2: track 10.8 -> 18.1 mm
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Other:
- outline, holes or cut-outs redrawn
- board text added: "1"
- board text added: "2"
- board text added: "34"
- board text added: "35"
- board text added: "36"
- board text added: "fNIRS UHD SiPM Splitter 2025-07 V1.0 ESH"
