File: KiCAD/sipm-hv-splitter/sipm-hv-splitter.kicad_pcb (KiCad board)
At the start: 6 copper layers, 63.5 x 33 mm, 133 parts, among them J1 Conn_02x18_Odd_Even, J2 Conn_02x17_Odd_Even, J3 -OMIT-, Q1 BSS138, Q2 BSS138, Q3 BSS138, U1 ATmega328-M, U10 OPA810xDCK, U11 OPA810xDCK, U12 OPA810xDCK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

Commit message: working on layout updates
Parts:
- added C54: 0.1uF, Capacitor_SMD:C_0603_1608Metric_Pad1.08x0.95mm_HandSolder, F.Cu at (86.5, 60.5)
- added C55: 0.1uF, Capacitor_SMD:C_0603_1608Metric_Pad1.08x0.95mm_HandSolder, F.Cu at (86.5, 56.8)
- added L2: 10uH, Inductor_SMD:L_0603_1608Metric_Pad1.05x0.95mm_HandSolder, F.Cu at (89.4, 62.0)
- J3: value -OMIT- -> ISP
- R16, R5: value 10.0k 1% -> 10.0k
- R6: value 10k -> 10.0k
- moved TP7 7.43 mm to (90.0, 49.1)
- moved R45 0.92 mm to (89.4, 56.8)
- moved R46 0.92 mm to (89.4, 58.5)
- moved R47 0.92 mm to (89.4, 55.0)
- moved C53 0.92 mm to (89.4, 60.3)
- moved D3 0.92 mm to (89.4, 53.0)
Connections:
- U1 pad 18: +3.3V -> Net-(U1-AVCC)
- U1 pad 20: unconnected-(U1-AREF-Pad20) -> Net-(U1-AREF)
Routing:
- net Net-(U1-PD2): track 10.7 -> 2.47 mm
- net /~{RESET}: track 12.2 -> 4.38 mm
- net Net-(U1-AVCC): track 0.00 -> 5.54 mm, vias 0 -> 1
- net /THERM: track 40.1 -> 36.5 mm
- net Net-(D3-A): track 2.77 -> 0.00 mm
- net Net-(U1-AREF): track 0.00 -> 2.72 mm
- net /ADC_VMON: track 17.3 -> 15.2 mm
- net GND: track 117.1 -> 118.9 mm, vias 78 -> 80
- net /MISO: track 34.0 -> 35.4 mm
- net /MOSI: track 27.8 -> 28.8 mm
- net /ADC_IMON: track 50.3 -> 49.7 mm

Commit message: Candidate V1.0 for review/fab
Parts:
- removed TP1: IMON, TestPoint:TestPoint_Pad_D1.0mm
- removed TP2: VIN60, TestPoint:TestPoint_Pad_D1.0mm
- removed TP3: CMP, TestPoint:TestPoint_Pad_D1.0mm
- removed TP4: VR_IN, TestPoint:TestPoint_Pad_D1.0mm
- removed TP5: VR_ADJ, TestPoint:TestPoint_Pad_D1.0mm
- removed TP6: DPOT, TestPoint:TestPoint_Pad_D1.0mm
- removed TP7: VSENSE, TestPoint:TestPoint_Pad_D1.0mm
Routing:
- net Net-(U1-PD2): track 2.47 -> 10.9 mm
- net /~{RESET}: track 4.38 -> 12.7 mm
- net /THERM: track 36.5 -> 39.7 mm
- net Net-(D3-A): track 0.00 -> 2.77 mm
- net /ADC_IMON: track 49.7 -> 47.3 mm
- net Net-(U5-A): track 5.97 -> 3.76 mm
- net Net-(Q2-G): track 40.9 -> 39.0 mm
Other:
- board text added: "SiPM BIAS BOARD V1.0 BACK ASSEMBLY"

Commit message: add mtg holes, L2 gnd fill
Parts:
- added H1: MountingHole, MountingHole:MountingHole_2.2mm_M2, F.Cu at (53.3, 53.3)
- added H2: MountingHole, MountingHole:MountingHole_2.2mm_M2, F.Cu at (53.3, 81.3)
- added H3: MountingHole, MountingHole:MountingHole_2.2mm_M2, F.Cu at (111.8, 81.3)
- added H4: MountingHole, MountingHole:MountingHole_2.2mm_M2, F.Cu at (111.8, 53.3)
Routing:
- net Net-(U1-AVCC): vias 1 -> 0
- added copper zone on In2.Cu, net GND
