File: KiCAD/sipm-hv-splitter/tia.kicad_sch (KiCad schematic)
At the start: 0 parts

Commit message: working on SiPM power supply schem
Parts:
- added C16, C24, C40: 0.1uF, Capacitor_SMD:C_0603_1608Metric_Pad1.08x0.95mm_HandSolder, symbol Device:C
- added C32: 1nF, Capacitor_SMD:C_0603_1608Metric_Pad1.08x0.95mm_HandSolder, symbol Device:C
- added R21: 4.7k, Resistor_SMD:R_0603_1608Metric_Pad0.98x0.95mm_HandSolder, symbol Device:R_US
- added R29: 15, Resistor_SMD:R_0603_1608Metric_Pad0.98x0.95mm_HandSolder, symbol Device:R_US
- added R37: 1k, Resistor_SMD:R_0603_1608Metric_Pad0.98x0.95mm_HandSolder, symbol Device:R_US
- added U6: OPA810xDCK, Package_TO_SOT_SMD:Texas_R-PDSO-G5_DCK-5, symbol Amplifier_Operational:OPA810xDCK
Connections:
- net VIN: now also R37.1
- net VOUT: now also R29.2
- new net: C32.1, C40.1, R21.1, R37.2, U6.4 (-)
- new net: C32.2, R21.2, R29.1, U6.1
- new net +3.3VA: C16.1, U6.5 (V+)
- new net -24V: C24.1, U6.2 (V-)
- new net GND: C16.2, C24.2, C40.2, U6.3 (+)

Commit message: routing madness
Parts:
- U6: footprint Package_TO_SOT_SMD:Texas_R-PDSO-G5_DCK-5 -> my_SC70:Texas_R-PDSO-G5_DCK-5
Changed lines of the file:
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@@
 			)
 		)
-		(property "Footprint" "Package_TO_SOT_SMD:Texas_R-PDSO-G5_DCK-5"
+		(property "Footprint" "my_SC70:Texas_R-PDSO-G5_DCK-5"
 			(at 87.376 97.028 0)
 			(effects

Commit message: working on bias filter changes
Parts:
- R21: value 4.7k -> 15k
Connections:
- net SIPM_A: now reaches C32.1, R21.1, U6.4 (-)
- net SIPM_A: no longer C40.1, R37.2
- net VIN renamed VBIAS
- new net SIPM_K: C40.1, R37.2
Other:
- note added: "SiPM Anode"
- note added: "SiPM Cathode"
- note added: "VBIAS in"
- moved on the sheet: C16, C24, C32, C40, R21, R29, R37, U6

Commit message: working on BOM
Parts:
- C16, C24, C40: CatNo (none) -> 311-1088-1-ND; MfgNo (none) -> CC0603KRX7R7BB104
- C32: CatNo (none) -> 1276-CL03B102KOSVPNCCT-ND; MfgNo (none) -> CL03B102KOSVPNC
- R37: CatNo (none) -> RMCF0603FT1K00CT-ND; MfgNo (none) -> RMCF0603FT1K00
Changed lines of the file:
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@@
+			)
+		)
+		(property "CatNo" "311-1088-1-ND"
+			(at 132.08 54.61 0)
+			(effects
+				(font
+					(size 1.27 1.27)
+				)
+				(hide yes)
+			)
+		)
+		(property "MfgNo" "CC0603KRX7R7BB104"
+			(at 132.08 54.61 0)
+			(effects
+				(font
+					(size 1.27 1.27)
+				)
+				(hide yes)
 			)
 		)
@@
 			)
 		)
+		(property "CatNo" "311-1088-1-ND"
+			(at 73.66 91.44 0)
+			(effects
+				(font
+					(size 1.27 1.27)
+				)
+				(hide yes)
+			)
+		)
+		(property "MfgNo" "CC0603KRX7R7BB104"
+			(at 73.66 91.44 0)
+			(effects
+				(font
+					(size 1.27 1.27)
+				)
+				(hide yes)
+			)
+		)
 		(pin "2"
 		)
@@
 			)
 		)
+		(property "CatNo" "RMCF0603FT1K00CT-ND"
+			(at 63.5 85.09 90)
+			(effects
+				(font
+					(size 1.27 1.27)
+				)
+				(hide yes)
+			)
+		)
+		(property "MfgNo" "RMCF0603FT1K00"
+			(at 63.5 85.09 90)
+			(effects
+				(font
+					(size 1.27 1.27)
+				)
+				(hide yes)
+			)
+		)
 		(pin "2"
 		)
@@
 		(property "Description" "Unpolarized capacitor"
 			(at 152.4 72.39 0)
+			(effects
+				(font
+					(size 1.27 1.27)
+				)
+				(hide yes)
+			)
+		)
+		(property "CatNo" "1276-CL03B102KOSVPNCCT-ND"
+			(at 152.4 72.39 90)
+			(effects
+				(font
+					(size 1.27 1.27)
+				)
+				(hide yes)
+			)
+		)
+		(property "MfgNo" "CL03B102KOSVPNC"
+			(at 152.4 72.39 90)
 			(effects
 				(font
@@
 			(at 132.08 99.06 0)
 			(effects
+				(font
+					(size 1.27 1.27)
+				)
+				(hide yes)
+			)
+		)
+		(property "CatNo" "311-1088-1-ND"
+			(at 132.08 99.06 0)
+			(effects
+				(font
+					(size 1.27 1.27)
+				)
+				(hide yes)
+			)
+		)
+		(property "MfgNo" "CC0603KRX7R7BB104"
+			(at 132.08 99.06 0)
+			(effects

Commit message: finish BOM entries on schematic
Parts:
- R21: CatNo (none) -> A121558CT-ND; MfgNo (none) -> CRG0603F15K
- R29: CatNo (none) -> 311-15.0HRCT-ND; MfgNo (none) -> RC0603FR-0715RL
- U6: CatNo (none) -> 296-OPA810IDCKRCT-ND; MfgNo (none) -> OPA810IDCKR
Changed lines of the file:
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@@
+			)
+		)
+		(property "CatNo" "A121558CT-ND"
+			(at 152.4 67.31 90)
+			(effects
+				(font
+					(size 1.27 1.27)
+				)
+				(hide yes)
+			)
+		)
+		(property "MfgNo" "CRG0603F15K"
+			(at 152.4 67.31 90)
+			(effects
+				(font
+					(size 1.27 1.27)
+				)
+				(hide yes)
 			)
 		)
@@
 			)
 		)
+		(property "CatNo" "311-15.0HRCT-ND"
+			(at 171.45 82.55 90)
+			(effects
+				(font
+					(size 1.27 1.27)
+				)
+				(hide yes)
+			)
+		)
+		(property "MfgNo" "RC0603FR-0715RL"
+			(at 171.45 82.55 90)
+			(effects
+				(font
+					(size 1.27 1.27)
+				)
+				(hide yes)
+			)
+		)
 		(pin "2"
 		)
@@
 			(effects
 				(font
+					(size 1.27 1.27)
+				)
+				(hide yes)
+			)
+		)
+		(property "CatNo" "296-OPA810IDCKRCT-ND"
+			(at 146.05 82.55 0)
+			(effects
+				(font
+					(size 1.27 1.27)
+				)
+				(hide yes)
+			)
+		)
+		(property "MfgNo" "OPA810IDCKR"
+			(at 146.05 82.55 0)
+			(effects
+				(font
