File: KiCAD/sipm-hv-splitter/sipm-hv-splitter.kicad_sch (KiCad schematic)
At the start: 17 parts, among them J1 Conn_02x18_Odd_Even, J2 Conn_02x17_Odd_Even, J3 -OMIT-, U1 ATmega328-M, U14 TPS7A25, U16 TPS7A25

Commit message: routing complete
Connections:
- net TIA_6/SIPM_K: now also J1.28 (Pin_28)
Changed lines of the file:
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@@
+	(wire
+		(pts
+			(xy 146.05 38.1) (xy 125.73 38.1)
+		)
+		(stroke
+			(width 0)
+			(type default)
+		)
+	)
 	(wire
 		(pts
@@
 	(wire
 		(pts
+			(xy 146.05 33.02) (xy 146.05 38.1)
+		)
+		(stroke
+			(width 0)
+			(type default)
+		)
+	)
+	(wire
+		(pts
 			(xy 125.73 63.5) (xy 140.97 63.5)
 		)
@@
 		)
 		(stroke
+			(width 0)
+			(type default)
+		)
+	)
+	(wire
+		(pts
+			(xy 162.56 33.02) (xy 146.05 33.02)
+		)
+		(stroke

Commit message: working on BOM
Parts:
- C48, C50, C52, C53: CatNo (none) -> 1276-1019-1-ND; MfgNo (none) -> CL10B105KO8NNNC
- C49, C51: CatNo (none) -> 587-2909-1-ND; MfgNo (none) -> TMK107ABJ225KA-T
- J3: value -OMIT- -> ISP
- R1: CatNo (none) -> RMCF0603FT1K00CT-ND; MfgNo (none) -> RMCF0603FT1K00
Changed lines of the file:
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@@
 			)
 		)
-		(property "Value" "-OMIT-"
+		(property "Value" "ISP"
 			(at 101.6 142.24 0)
 			(effects
@@
 			)
 		)
+		(property "CatNo" "587-2909-1-ND"
+			(at 241.3 137.16 0)
+			(effects
+				(font
+					(size 1.27 1.27)
+				)
+				(hide yes)
+			)
+		)
+		(property "MfgNo" "TMK107ABJ225KA-T"
+			(at 241.3 137.16 0)
+			(effects
+				(font
+					(size 1.27 1.27)
+				)
+				(hide yes)
+			)
+		)
 		(pin "1"
 		)
@@
 			)
 		)
+		(property "CatNo" "1276-1019-1-ND"
+			(at 167.64 137.16 0)
+			(effects
+				(font
+					(size 1.27 1.27)
+				)
+				(hide yes)
+			)
+		)
+		(property "MfgNo" "CL10B105KO8NNNC"
+			(at 167.64 137.16 0)
+			(effects
+				(font
+					(size 1.27 1.27)
+				)
+				(hide yes)
+			)
+		)
 		(pin "1"
 		)
@@
 			)
 		)
+		(property "CatNo" "1276-1019-1-ND"
+			(at 101.6 77.47 0)
+			(effects
+				(font
+					(size 1.27 1.27)
+				)
+				(hide yes)
+			)
+		)
+		(property "MfgNo" "CL10B105KO8NNNC"
+			(at 101.6 77.47 0)
+			(effects
+				(font
+					(size 1.27 1.27)
+				)
+				(hide yes)
+			)
+		)
 		(pin "1"
 		)
@@
 			)
 		)
+		(property "CatNo" "1276-1019-1-ND"
+			(at 57.15 96.52 0)
+			(effects
+				(font
+					(size 1.27 1.27)
+				)
+				(hide yes)
+			)
+		)
+		(property "MfgNo" "CL10B105KO8NNNC"
+			(at 57.15 96.52 0)
+			(effects
+				(font
+					(size 1.27 1.27)
+				)
+				(hide yes)
+			)
+		)
 		(pin "1"
 		)
@@
 			)
 		)
+		(property "CatNo" "587-2909-1-ND"
+			(at 196.85 135.89 0)
+			(effects
+				(font
+					(size 1.27 1.27)
+				)
+				(hide yes)
+			)
+		)
+		(property "MfgNo" "TMK107ABJ225KA-T"
+			(at 196.85 135.89 0)
+			(effects
+				(font
+					(size 1.27 1.27)
+				)
+				(hide yes)
+			)
+		)
 		(pin "1"
 		)
@@
 		(property "Description" "Resistor, US symbol"
 			(at 224.79 77.47 0)
+			(effects
+				(font
+					(size 1.27 1.27)
+				)
+				(hide yes)
+			)
+		)
+		(property "CatNo" "RMCF0603FT1K00CT-ND"
+			(at 224.79 77.47 90)
+			(effects
+				(font
+					(size 1.27 1.27)
+				)
+				(hide yes)
+			)
+		)
+		(property "MfgNo" "RMCF0603FT1K00"
+			(at 224.79 77.47 90)
 			(effects
 				(font
@@
 			(at 210.82 137.16 0)
 			(effects
+				(font
+					(size 1.27 1.27)
+				)
+				(hide yes)
+			)
+		)
+		(property "CatNo" "1276-1019-1-ND"
+			(at 210.82 137.16 0)
+			(effects
+				(font
+					(size 1.27 1.27)
+				)
+				(hide yes)
+			)
+		)
+		(property "MfgNo" "CL10B105KO8NNNC"
+			(at 210.82 137.16 0)
+			(effects

Commit message: finish BOM entries on schematic
Parts:
- R45: MfgNo (none) -> ERJ-3EKF4701V
- R46: CatNo P4.70KHCT-ND -> 311-10.0KHRCT-ND; MfgNo (none) -> CRCW0603100KFKEA
- U1: CatNo (none) -> ATMEGA328P-MU-ND; MfgNo (none) -> ATMEGA328P-MU
- U14, U16: CatNo (none) -> 296-TPS7A2533DRVRCT-ND; MfgNo (none) -> TPS7A2533DRVR
Changed lines of the file:
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@@
+			)
+		)
+		(property "CatNo" "296-TPS7A2533DRVRCT-ND"
+			(at 182.88 133.35 0)
+			(effects
+				(font
+					(size 1.27 1.27)
+				)
+				(hide yes)
+			)
+		)
+		(property "MfgNo" "TPS7A2533DRVR"
+			(at 182.88 133.35 0)
+			(effects
+				(font
+					(size 1.27 1.27)
+				)
+				(hide yes)
 			)
 		)
@@
 			)
 		)
+		(property "MfgNo" "ERJ-3EKF4701V"
+			(at 132.08 129.54 0)
+			(effects
+				(font
+					(size 1.27 1.27)
+				)
+				(hide yes)
+			)
+		)
 		(pin "1"
 		)
@@
 			)
 		)
+		(property "CatNo" "ATMEGA328P-MU-ND"
+			(at 46.99 140.97 0)
+			(effects
+				(font
+					(size 1.27 1.27)
+				)
+				(hide yes)
+			)
+		)
+		(property "MfgNo" "ATMEGA328P-MU"
+			(at 46.99 140.97 0)
+			(effects
+				(font
+					(size 1.27 1.27)
+				)
+				(hide yes)
+			)
+		)
 		(pin "8"
 		)
@@
 			)
 		)
-		(property "CatNo" "P4.70KHCT-ND"
+		(property "CatNo" "311-10.0KHRCT-ND"
 			(at 101.6 67.31 0)
 			(effects
@@
 		)
 		(property "Vendor" "DigiKey"
+			(at 101.6 67.31 0)
+			(effects
+				(font
+					(size 1.27 1.27)
+				)
+				(hide yes)
+			)
+		)
+		(property "MfgNo" "CRCW0603100KFKEA"
 			(at 101.6 67.31 0)
 			(effects
@@
 			(at 226.06 133.35 0)
 			(effects
+				(font
+					(size 1.27 1.27)
+				)
+				(hide yes)
+			)
+		)
+		(property "CatNo" "296-TPS7A2533DRVRCT-ND"
+			(at 226.06 133.35 0)
+			(effects
+				(font
+					(size 1.27 1.27)
+				)
+				(hide yes)
+			)
+		)
+		(property "MfgNo" "TPS7A2533DRVR"
+			(at 226.06 133.35 0)
+			(effects

Commit message: working on layout updates
Parts:
- added C54, C55: 0.1uF, Capacitor_SMD:C_0603_1608Metric_Pad1.08x0.95mm_HandSolder, symbol Device:C
- added L2: 10uH, Inductor_SMD:L_0603_1608Metric_Pad1.05x0.95mm_HandSolder, symbol Device:L
Connections:
- net +3.3V: now also L2.1; no longer U1.18 (AVCC)
- net GND: now also C54.2, C55.2
- net at U1.20 (AREF): now also C55.1
- new net: C54.1, L2.2, U1.18 (AVCC)
Other:
- moved on the sheet: C52

Commit message: add temperature readout
Other:
- note added: "BLK"
- note added: "RED"
- note added: "SHD"
- note added: "WHT"
Changed lines of the file:
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@@
+		)
+	)
+	(text "WHT"
+		(exclude_from_sim no)
+		(at 106.68 35.052 0)
+		(effects
+			(font
+				(size 1.27 1.27)
+			)
+		)
+	)
+	(text "RED"
+		(exclude_from_sim no)
+		(at 139.7 32.004 0)
+		(effects
+			(font
+				(size 1.27 1.27)
+			)
+		)
+	)
+	(text "BLK"
+		(exclude_from_sim no)
+		(at 139.7 34.798 0)
+		(effects
+			(font
+				(size 1.27 1.27)
+			)
 		)
 	)
@@
 		)
 	)
+	(text "SHD"
+		(exclude_from_sim no)
+		(at 106.426 32.004 0)
+		(effects
+			(font
+				(size 1.27 1.27)
+			)
+		)
+	)
 	(text "ISP Header (1mm)\n(same as on IMU\nfor which we have\nan adapter PCB)"
 		(exclude_from_sim no)
@@
 		)
 		(stroke
+			(width 0)
+			(type default)
+		)
+	)
+	(wire
+		(pts
+			(xy 104.14 35.56) (xy 113.03 35.56)
+		)
+		(stroke
