File: NN26_27/Electronics/SrcInterfaceCard/NN22_VCCS_SrcAdapter02_s00.sch (EAGLE design)
At the start: 146 parts, among them J1 M04X2_0.050_SMD_NO_CREAM, J2 M13X2_0.050_SHF, J3 M04X2_0.050_SMD_NO_CREAM, J4 U.FL, J5 M20X2_HARFLEX_M, J6 M03X1_JST_SH_RA, J7 USB-MICRO, Q1 MOSFET-DUAL-N-UDFN8, Q10 MOSFET-DUAL-N-UDFN8, Q2 MOSFET-DUAL-N-UDFN8, Q3 MOSFET-DUAL-N-UDFN8, Q4 MOSFET-DUAL-N-UDFN8, Q5 MOSFET-DUAL-N-UDFN8, Q6 MOSFET-DUAL-N-UDFN8, Q7 MOSFET-DUAL-N-UDFN8, Q8 MOSFET-DUAL-N-UDFN8, Q9 MOSFET-DUAL-N-UDFN8, U1 74HC238_TSSOP, U10 LDL212_DFN6_3X3, U2 74HC238_TSSOP, U3 AD5683R_MSOP, U4 OPA392_SOT23, U5 RP2040, U6 W25Q_USON, U7 ADP7182_WSON, U8 MCP1755_DFN, U9 LDL212_DFN6_3X3, X1 CRYSTAL-3.2-2.5

Commit message: Adding NN26 upgrade notes.
Other:
- note added: "Configuration for high power source optodes: R9: 1 Ohm R13: 2.2 Ohm C12: 0.22 uF R8: 1.5 Ohm R30: 59 kOhm F1: 0ZCH0110AF2E R2: 12 kOhm"
- note removed: "Configuration for high power source optodes: R9: 1 Ohm R13: 2.2 Ohm C12: 0.22 uF R8: 1.5 Ohm R30: 56k Ohm (better would be ~59k) F1: 0ZCH0110AF2E R2: 12k Ohm"
Changed lines of the file:
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@@
 C12: 0.22 uF
 R8: 1.5 Ohm
-R30: 56k Ohm (better would be ~59k)
+R30: 59 kOhm
 F1: 0ZCH0110AF2E
-R2: 12k Ohm</text>
+R2: 12 kOhm</text>
 </plain>
 <instances>
@@
 C12: 0.22 uF
 R8: 1.5 Ohm
-R30: 56k Ohm (better would be ~59k)
+R30: 59 kOhm
 F1: 0ZCH0110AF2E
-R2: 12k Ohm</text>
+R2: 12 kOhm</text>
 </plain>
 <instances>
