File: NN26_27/Electronics/DetInterfaceCard/DetAdapter03_KiCAD/NN22_RPi_DetAdapter03_s00.kicad_pcb (KiCad board)
At the start: 6 copper layers, 63.5 x 33 mm, 239 parts, among them J1 M17X2, J2 M05X2_SMD_0.050_NOCREAM, J3 M03X1_0.050_SMD_NO_CREAM, J4 USB-MICRO, J5 M20X2_HARFLEX_M, U1 AD7380, U10 RP2040, U11 MCP1755_DFN, U12 MCP1755_DFN, U13 ADP7142_WSON, U14 ADP7182_WSON, U15 ADP7182_WSON, U2 ADA4940-2, U3 AD7380, U4 ADA4940-2, U5 AD7380, U6 ADA4940-2, U7 AD7380, U8 ADA4940-2, U9 W25Q_USON_PAD, X1 CRYSTAL-3.2-2.5

Commit message: change diode footprint
Parts:
- D1, D2: value SBR1A20T5 -> SBR1U40LP; footprint SOD523 -> my_DFN:DFN1411
- LED1: value (none) -> LED0603
- moved D1 0.54 mm to (169.8, 93.0), turned to 90 degrees
- moved D2 0.31 mm to (167.0, 95.6), turned to -90 degrees
Connections:
- net /CS_A1 renamed /CS_A1
- net /CS_A2 renamed /CS_A2
- net /CS_A3 renamed /CS_A3
- net /CS_A4 renamed /CS_A4
- net V6P5CON renamed Net-(LF1-P$1)
- net VN20P0CON renamed Net-(LF2-P$1)
- J1 pad 34: (no net) -> unconnected-(J1-Pad34)
- J4 pad 4: (no net) -> unconnected-(J4-Pad4)
- U11 pad 2: (no net) -> unconnected-(U11-PWRGD-Pad2)
- U12 pad 2: (no net) -> unconnected-(U12-PWRGD-Pad2)
- U13 pad 5: (no net) -> unconnected-(U13-SS-Pad5)
- U2 pad 14: (no net) -> unconnected-(U2B-/DISABLE-Pad14)
- U2 pad 20: (no net) -> unconnected-(U2A-/DISABLE-Pad20)
- U4 pad 14: (no net) -> unconnected-(U4B-/DISABLE-Pad14)
- U4 pad 20: (no net) -> unconnected-(U4A-/DISABLE-Pad20)
- U6 pad 14: (no net) -> unconnected-(U6B-/DISABLE-Pad14)
- U6 pad 20: (no net) -> unconnected-(U6A-/DISABLE-Pad20)
- U8 pad 14: (no net) -> unconnected-(U8B-/DISABLE-Pad14)
- U8 pad 20: (no net) -> unconnected-(U8A-/DISABLE-Pad20)
Routing:
- net V5P0: track 21.3 -> 21.8 mm
Other:
- board text added: "NinjaNIRS 2026 Detector Interface v03a 08/2026"
- board text added: "V03A"
- board text removed: "NinjaNIRS 2026 Detector Interface v03 07/2026"
