File: NN26_27/Electronics/DetInterfaceCard/DetAdapter03_KiCAD/NN22_RPi_DetAdapter03_s00.kicad_sch (KiCad schematic)
At the start: 46 parts, among them J1 M17X2, U1 AD7380, U2 ADA4940-2

Commit message: update schematic to include MPN1, MFG1
Parts:
- C1, C11, C18, C5: MFG1 (none) -> Murata; MPN1 (none) -> GRM1555C1H331JA01D
- C10, C13, C19, C20, C21, C8, C9: MFG1 (none) -> Murata; MPN1 (none) -> GRM155R71H104KE14D
- C12, C14, C6, C7: MFG1 (none) -> Samsung; MPN1 (none) -> CL05A105KP5NNNC
- C15, C16, C17, C2, C3, C4: MFG1 (none) -> Murata; MPN1 (none) -> GRM1555C1H102JA01D
- J1: MFG1 (none) -> Samtec; MPN1 (none) -> SHF-117-01-L-D-SM
- LF1, LF2: MFG1 (none) -> Murata; MPN1 (none) -> BLM18AG601SN1D
- R1, R10, R13, R14, R4, R7: MFG1 (none) -> Susumu; MPN1 (none) -> RR0510P-183-D
- R11, R2, R5, R8: MFG1 (none) -> Susumu; MPN1 (none) -> RR0510P-222-D
- R12, R3, R6, R9: MFG1 (none) -> Vishay; MPN1 (none) -> CRCW040233R0FKEDC
- R71, TP1, TP2, TP3, TP4, TP5: now not fitted
- U1: MFG1 (none) -> Analog Devices; MPN1 (none) -> AD7380BCPZ-RL7
- U2: MFG1 (none) -> Analog Devices; MPN1 (none) -> ADA4940-2ACPZ-R7
