File: NN26_27/Electronics/DetInterfaceCard/DetAdapter03_KiCAD/NN22_RPi_DetAdapter03_s00_2.kicad_sch (KiCad schematic)
At the start: 40 parts, among them U3 AD7380, U4 ADA4940-2

Commit message: update schematic to include MPN1, MFG1
Parts:
- C22, C26, C32, C39: MFG1 (none) -> Murata; MPN1 (none) -> GRM1555C1H331JA01D
- C23, C24, C25, C36, C37, C38: MFG1 (none) -> Murata; MPN1 (none) -> GRM1555C1H102JA01D
- C27, C28, C33, C35: MFG1 (none) -> Samsung; MPN1 (none) -> CL05A105KP5NNNC
- C29, C30, C31, C34, C40, C41, C42: MFG1 (none) -> Murata; MPN1 (none) -> GRM155R71H104KE14D
- R15, R18, R21, R24, R27, R28: MFG1 (none) -> Susumu; MPN1 (none) -> RR0510P-183-D
- R16, R19, R22, R25: MFG1 (none) -> Susumu; MPN1 (none) -> RR0510P-222-D
- R17, R20, R23, R26: MFG1 (none) -> Vishay; MPN1 (none) -> CRCW040233R0FKEDC
- TP6, TP7, TP8: now not fitted
- U3: MFG1 (none) -> Analog Devices; MPN1 (none) -> AD7380BCPZ-RL7
- U4: MFG1 (none) -> Analog Devices; MPN1 (none) -> ADA4940-2ACPZ-R7
