File: NN26_27/Electronics/DetInterfaceCard/DetAdapter03_KiCAD/NN22_RPi_DetAdapter03_s00_3.kicad_sch (KiCad schematic)
At the start: 41 parts, among them J2 M05X2_SMD_0.050_NOCREAM, U5 AD7380, U6 ADA4940-2

Commit message: update schematic to include MPN1, MFG1
Parts:
- C43, C47, C53, C60: MFG1 (none) -> Murata; MPN1 (none) -> GRM1555C1H331JA01D
- C44, C45, C46, C57, C58, C59: MFG1 (none) -> Murata; MPN1 (none) -> GRM1555C1H102JA01D
- C48, C49, C54, C56: MFG1 (none) -> Samsung; MPN1 (none) -> CL05A105KP5NNNC
- C50, C51, C52, C55, C61, C62, C63: MFG1 (none) -> Murata; MPN1 (none) -> GRM155R71H104KE14D
- J2, TP11, TP12, TP9: now not fitted
- R29, R32, R35, R38, R41, R42: MFG1 (none) -> Susumu; MPN1 (none) -> RR0510P-183-D
- R30, R33, R36, R39: MFG1 (none) -> Susumu; MPN1 (none) -> RR0510P-222-D
- R31, R34, R37, R40: MFG1 (none) -> Vishay; MPN1 (none) -> CRCW040233R0FKEDC
- U5: MFG1 (none) -> Analog Devices; MPN1 (none) -> AD7380BCPZ-RL7
- U6: MFG1 (none) -> Analog Devices; MPN1 (none) -> ADA4940-2ACPZ-R7
