File: NN26_27/Electronics/DetInterfaceCard/DetAdapter03_KiCAD/NN22_RPi_DetAdapter03_s00_4.kicad_sch (KiCad schematic)
At the start: 40 parts, among them U7 AD7380, U8 ADA4940-2

Commit message: update schematic to include MPN1, MFG1
Parts:
- C64, C68, C74, C81: MFG1 (none) -> Murata; MPN1 (none) -> GRM1555C1H331JA01D
- C65, C66, C67, C78, C79, C80: MFG1 (none) -> Murata; MPN1 (none) -> GRM1555C1H102JA01D
- C69, C70, C75, C77: MFG1 (none) -> Samsung; MPN1 (none) -> CL05A105KP5NNNC
- C71, C72, C73, C76, C82, C83, C84: MFG1 (none) -> Murata; MPN1 (none) -> GRM155R71H104KE14D
- R43, R46, R49, R52, R55, R56: MFG1 (none) -> Susumu; MPN1 (none) -> RR0510P-183-D
- R44, R47, R50, R53: MFG1 (none) -> Susumu; MPN1 (none) -> RR0510P-222-D
- R45, R48, R51, R54: MFG1 (none) -> Vishay; MPN1 (none) -> CRCW040233R0FKEDC
- TP13, TP15, TP16: now not fitted
- U7: MFG1 (none) -> Analog Devices; MPN1 (none) -> AD7380BCPZ-RL7
- U8: MFG1 (none) -> Analog Devices; MPN1 (none) -> ADA4940-2ACPZ-R7
