File: NN26_27/Electronics/DetInterfaceCard/DetAdapter03_KiCAD/NN22_RPi_DetAdapter03_s00_5.kicad_sch (KiCad schematic)
At the start: 19 parts, among them J3 M03X1_0.050_SMD_NO_CREAM, J4 USB-MICRO, J5 M20X2_HARFLEX_M, U10 RP2040, U9 W25Q_USON_PAD, X1 CRYSTAL-3.2-2.5

Commit message: update schematic to include MPN1, MFG1
Parts:
- C85: MFG1 (none) -> Murata; MPN1 (none) -> GRM155R71H104KE14D
- C86, C87: MFG1 (none) -> Murata; MPN1 (none) -> GCM1555C1H270JA16D
- J3, R63: now not fitted
- J4: MFG1 (none) -> Amphenol Communications Solutions; MPN1 (none) -> 101181940001LF
- J5: MFG1 (none) -> HARTING Elektronik; MPN1 (none) -> 15150402601000
- LED1: MFG1 (none) -> Lite-On; MPN1 (none) -> LTST-C191KRKT
- R57, R62, R64: MFG1 (none) -> Yageo; MPN1 (none) -> RC0402FR-071K2L
- R58, R59: MFG1 (none) -> Yageo; MPN1 (none) -> RC0402FR-07100KL
- R60, R61: MFG1 (none) -> Yageo; MPN1 (none) -> RC0402FR-0727RL
- S1: MFG1 (none) -> C&K Components; MPN1 (none) -> KMR231NGLFS
- U10: MFG1 (none) -> Raspberry Pi; MPN1 (none) -> SC0914(7)
- U9: MFG1 (none) -> Winbond; MPN1 (none) -> W25Q16RVXHJQ TR
- X1: MFG1 (none) -> CTS Components; MPN1 (none) -> 403I35D12M00000
